File: board.brd (EAGLE design)
At the start: 26.3 x 33.6 mm, 46 parts, among them IC1 ATMEGA48/88/168-AU, IC2 TP4056, IC3 MAX31865, IC4 MCP1703CB, Q1 PH2925U, Q2 IRLML2244

Commit message: draft
Parts:
- removed C5, C6: 100n, rcl:C0603
- removed GND_LED: (no value), wirepad:SMD1,27-2,54
- removed IC3: MAX31865, Oles komponentbibliotek:TQFN20-5X5
- removed R2, R3: 200, rcl:R0603
- removed XTAL: (no value), xtal:CS10
- added MISO, MOSI, RST, SCK, VCC_LED: (no value), wirepad:SMD1,27-2,54
- Q2: value IRLML2244 -> CSTCR6M00G53Z; device SparkFun-DiscreteSemi:SOT23-3 -> murata-filter:CSTCR6M
- R4: value 10k -> 500
- moved RTD1 83.3 mm to (-48.3, -10.2)
- moved RTD2 77.9 mm to (-44.5, -10.2)
- moved R4 74.8 mm to (-49.5, -16.5), turned to 0 degrees
- moved C4 70.8 mm to (-47.0, 31.8), turned to 0 degrees
- moved R1 60.6 mm to (-31.8, 43.2)
- moved R8 60.3 mm to (-49.5, 38.1), turned to 0 degrees
- moved C10 60.3 mm to (-30.5, 38.1), turned to 0 degrees
- moved R9 56.6 mm to (-41.9, 43.2)
- moved GND 54.1 mm to (-33.0, 31.8)
- moved IC1 54.0 mm to (16.5, 64.8)
- moved C3 53.7 mm to (-40.6, 31.8), turned to 0 degrees
- moved R7 53.4 mm to (-43.2, 38.1), turned to 0 degrees
- moved C11 52.2 mm to (-36.8, 38.1)
- moved Q2 50.8 mm to (24.1, 68.6), turned to 90 degrees
- moved R11 46.2 mm to (-16.5, 43.2)
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Connections:
- removed net D10_CS: IC1.14, IC3.13
- removed net D2_BUTTON: BTN1.1, IC1.32
- removed net D5_LED1: IC1.9, R5.2
- removed net D6_LED2: IC1.10, R6.2
- removed net D8_VCC_MAX: IC1.12, Q2.1, R4.1
- removed net D9_LED3: IC1.13, R12.2
- removed net N$5: R2.1, R3.2
- removed net TEMP_IN-: C6.2, IC3.8, IC3.9, RTD2.1
- removed net TEMP_REF+: IC3.1, IC3.2, R2.2
- removed net TEMP_REF-: IC3.3, IC3.4, R3.1
- removed net VCC_MAX: C5.1, IC3.19, IC3.20, Q2.3
- removed net XTAL2: IC1.8, XTAL.L
- new net D10_LED3: IC1.14, R12.2
- new net D2: IC1.32
- new net D5_TEMP: IC1.9
- new net D6: IC1.10
- new net D8_LED1: IC1.12, R5.2
- new net D9_LED2: IC1.13, R6.2
- new net N$1: IC1.8, Q2.3
- new net N$2: RTD2.1
- net D11_MOSI: now also MOSI.1; no longer IC3.11
- net D12_MISO: now also MISO.1; no longer IC3.14
- net D13_SCK: now also SCK.1; no longer IC3.12
- net GND: now also Q2.2; no longer BTN2.1, C5.2, GND_LED.1, IC3.10, IC3.15, IC3.16, IC3.6, IC3.EXP, R4.2
- net RST: now also RST.1
- net TEMP_IN+: now also R4.2; no longer C6.1, IC3.5, IC3.7
- net VBAT: now also BTN2.1; no longer BAT+.1
- net VCC: now also BAT+.1, BTN1.1, R4.1, VCC_LED.1; no longer Q2.2
- net XTAL1: now also Q2.1; no longer XTAL.R
Routing:
- net VCC: track 47.5 -> 0.00 mm, vias 4 -> 0
- net D3_GATE: track 23.8 -> 0.00 mm, vias 2 -> 0
- net D6_LED2: track 16.8 -> 0.00 mm, vias 2 -> 0
- net D5_LED1: track 16.6 -> 0.00 mm, vias 2 -> 0
- net VBAT: track 15.4 -> 0.00 mm
- net D13_SCK: track 14.4 -> 0.00 mm
- net D11_MOSI: track 14.4 -> 0.00 mm, vias 2 -> 0
- net D10_CS: track 13.8 -> 0.00 mm, vias 2 -> 0
- net A0_CHRG_EN: track 13.6 -> 0.00 mm, vias 2 -> 0
- net D9_LED3: track 13.6 -> 0.00 mm, vias 2 -> 0
- net A2_CHRG_STBY: track 12.5 -> 0.00 mm, vias 2 -> 0
- net A1_CHRG_STAT: track 12.1 -> 0.00 mm, vias 2 -> 0
- net A7_VSENS: track 12.1 -> 0.00 mm
- net COIL: track 11.0 -> 0.00 mm, vias 9 -> 0
- net D12_MISO: track 11.0 -> 0.00 mm
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- removed copper zone on layer 1, net GND
- removed copper zone on layer 16, net GND
Other:
- board size 26.3 x 33.6 mm -> 100 x 80 mm
- board text removed: "Vapoduino_v0.2"
